Commit message: fix: stabilize simulation launch, moveit semantics, and force estimation

File: cobot_description/urdf/cobot.xacro (robot description, xacro)
@@ -5,4 +5,5 @@
    <xacro:arg name="sim_gazebo" default="false" />
    <xacro:arg name="use_soem" default="false" />
+   <xacro:arg name="use_modular_hardware" default="false" />
    <xacro:arg name="initial_mode_of_operation" default="8" />
    <xacro:include filename="$(find cobot_description)/urdf/cobot_arm.xacro"/>
@@ -19,4 +20,10 @@
          <material name="blue"/>
       </visual>
+      <collision>
+         <origin xyz="0 0 0" rpy="0 0 0"/>
+         <geometry>
+            <box size="0.02 0.02 0.02"/>
+         </geometry>
+      </collision>
       <inertial>
          <mass value="0.001"/>
@@ -50,4 +57,5 @@
       sim_gazebo="$(arg sim_gazebo)"
       use_soem="$(arg use_soem)"
+      use_modular_hardware="$(arg use_modular_hardware)"
       initial_mode_of_operation="$(arg initial_mode_of_operation)" />
 </robot>

File: cobot_description/urdf/cobot_arm.xacro (robot description, xacro)
@@ -201,4 +201,6 @@
             </inertial>
         </link>
+        <!-- Legacy TCP (Commented out to prevent conflict with gripper_tcp) -->
+        <!--
         <joint name="eef_tcp" type="fixed">
             <parent link="link_6" />
@@ -207,4 +209,5 @@
         </joint>
         <link name="eef_tcp_link" />
+        -->
     </xacro:macro>
 </robot>

File: cobot_description/urdf/cobot_ros2_control.xacro (robot description, xacro)
@@ -5,4 +5,5 @@
     sim_gazebo:=false
     use_soem:=false
+    use_modular_hardware:=false
     initial_mode_of_operation:=8
     ">
@@ -106,5 +107,5 @@
     <xacro:if value="${sim_gazebo}">
       <gazebo>
-        <plugin filename="libgz_ros2_control-system.so" name="gz_ros2_control::GazeboSimROS2ControlPlugin">
+        <plugin filename="ign_ros2_control-system" name="ign_ros2_control::IgnitionROS2ControlPlugin">
           <parameters>$(find cobot_description)/config/cobot_controllers.yaml</parameters>
         </plugin>
@@ -126,5 +127,18 @@
           <param name="control_frequency">1000</param>
         </xacro:if>
-        <xacro:if value="${not (sim_gazebo or use_fake_hardware or use_soem)}">
+        <xacro:if value="${use_modular_hardware}">
+          <plugin>cobot_hardware/ViroHardware</plugin>
+          <param name="port">/tmp/ttyViro</param>
+          <param name="baud">115200</param>
+          <sensor name="wrist_ft_sensor">
+            <state_interface name="force.x"/>
+            <state_interface name="force.y"/>
+            <state_interface name="force.z"/>
+            <state_interface name="torque.x"/>
+            <state_interface name="torque.y"/>
+            <state_interface name="torque.z"/>
+          </sensor>
+        </xacro:if>
+        <xacro:if value="${not (sim_gazebo or use_fake_hardware or use_soem or use_modular_hardware)}">
           <plugin>ethercat_driver/EthercatDriver</plugin>
           <param name="master_id">0</param>
@@ -134,4 +148,7 @@
       <joint name="joint_1">
         <command_interface name="reset_fault"/>
+        <xacro:if value="${use_modular_hardware}">
+          <param name="node_id">1</param>
+        </xacro:if>
         <xacro:if value="${initial_mode_of_operation == 8 or initial_mode_of_operation == '8'}">
           <command_interface name="position">
@@ -159,4 +176,7 @@
       <joint name="joint_2">
         <command_interface name="reset_fault"/>
+        <xacro:if value="${use_modular_hardware}">
+          <param name="node_id">2</param>
+        </xacro:if>
         <xacro:if value="${initial_mode_of_operation == 8 or initial_mode_of_operation == '8'}">
           <command_interface name="position">
@@ -184,4 +204,7 @@
       <joint name="joint_3">
         <command_interface name="reset_fault"/>
+        <xacro:if value="${use_modular_hardware}">
+          <param name="node_id">3</param>
+        </xacro:if>
         <xacro:if value="${initial_mode_of_operation == 8 or initial_mode_of_operation == '8'}">
           <command_interface name="position">
@@ -209,4 +232,7 @@
       <joint name="joint_4">
         <command_interface name="reset_fault"/>
+        <xacro:if value="${use_modular_hardware}">
+          <param name="node_id">4</param>
+        </xacro:if>
         <xacro:if value="${initial_mode_of_operation == 8 or initial_mode_of_operation == '8'}">
           <command_interface name="position">
@@ -234,4 +260,7 @@
       <joint name="joint_5">
         <command_interface name="reset_fault"/>
+        <xacro:if value="${use_modular_hardware}">
+          <param name="node_id">5</param>
+        </xacro:if>
         <xacro:if value="${initial_mode_of_operation == 8 or initial_mode_of_operation == '8'}">
           <command_interface name="position">
@@ -259,4 +288,7 @@
       <joint name="joint_6">
         <command_interface name="reset_fault"/>
+        <xacro:if value="${use_modular_hardware}">
+          <param name="node_id">6</param>
+        </xacro:if>
         <xacro:if value="${initial_mode_of_operation == 8 or initial_mode_of_operation == '8'}">
           <command_interface name="position">
